Commit message: update urdf with lidar

File: src/S10_sdk_deploy/S10_description/s10_mjcf/urdf/S10.urdf (robot description, URDF)
Before this commit: robot S10, 18 links, 17 joints
Links:
- added link back_lidar_link
- added link front_lidar_link
Joints:
- added joint back_lidar_joint: type fixed, parent base_link, child back_lidar_link, origin xyz=-0.22341 0.0 -0.0001 rpy=0 0 3.14159
- added joint front_lidar_joint: type fixed, parent base_link, child front_lidar_link, origin xyz=0.22341 0.0 -0.0001 rpy=0 0 0
